Commit message: final commit

File: resource/2DrobotArm/robot_3D.urdf (robot description, URDF)
Before this commit: robot 2DrobotArm, 5 links, 4 joints
Joints:
- removed joint link1Tolink3
- added joint link2Tolink3: type revolute, parent link2, child link3, origin xyz=0 0 0.3, axis 1 0 0

File: resource/aliengo/aliengo_modified.urdf (robot description, URDF)
Before this commit: robot aliengo_description, 19 links, 18 joints
Joints:
- joint RR_thigh_joint: type continuous -> revolute
